Commit message: WIP: switched to ros2_control and scout mini robot

File: scout_ros2/scout_description/urdf/scout_mini/scout_mini.xacro (robot description, xacro)
@@ -26,5 +26,22 @@
     <xacro:property name="imu_offset_y" value="0"/>
     <xacro:property name="imu_offset_z" value="${-base_z_size/2 + 0.005 + 0.007}"/>
-    <!-- Base link -->
+    <!-- Dummy Root Link -->
+    <link name="dummy_base_link">
+        <!-- No inertial properties for the root link -->
+        <visual>
+            <geometry>
+                <box size="0.001 0.001 0.001" />
+            </geometry>
+            <material name="transparent">
+                <color rgba="0 0 0 0" />
+            </material>
+        </visual>
+        <collision>
+            <geometry>
+                <box size="0.001 0.001 0.001" />
+            </geometry>
+        </collision>
+    </link>
+    <!-- Base Link -->
     <link name="base_link">
         <visual>
@@ -46,4 +63,10 @@
         </inertial>
     </link>
+    <!-- Joint connecting dummy_base_link to base_link -->
+    <joint name="dummy_to_base_joint" type="fixed">
+        <parent link="dummy_base_link" />
+        <child link="base_link" />
+        <origin xyz="0 0 0" rpy="0 0 0" />
+    </joint>
     <link name="base_footprint"/>
     <joint name="base_footprint_joint" type="fixed">
@@ -152,5 +175,5 @@
             <update_rate>100</update_rate>
             <visualize>false</visualize>
-            <topic>/model/scout_mini/imu</topic>
+            <topic>/model/robot/imu</topic>
             <frame_id>imu</frame_id>
             <gz_frame_id>imu</gz_frame_id>
@@ -161,5 +184,5 @@
         <sensor name="laser2d" type="gpu_lidar">
             <pose relative_to="laser2d">0 0 0 0 0 0</pose>
-            <topic>/model/scout_mini/scan</topic>
+            <topic>/model/robot/scan</topic>
             <update_rate>10</update_rate>
             <ray>
@@ -194,5 +217,5 @@
         <sensor name="laser3d" type="gpu_lidar">
             <pose relative_to="laser3d">0 0 0 0 0 0</pose>
-            <topic>/model/scout_mini/cloud</topic>
+            <topic>/model/robot/cloud</topic>
             <update_rate>10</update_rate>
             <ray>
@@ -226,51 +249,4 @@
     <gazebo>
         <plugin
-            filename="libignition-gazebo-diff-drive-system.so"
-            name="ignition::gazebo::systems::DiffDrive">
-            <num_wheel_pairs>2</num_wheel_pairs>
-            <!-- wheels0 -->
-            <left_joint>front_left_wheel</left_joint>
-            <right_joint>front_right_wheel</right_joint>
-            <wheel_separation>${track}</wheel_separation>
-            <wheel_radius>${wheel_radius}</wheel_radius>
-            <!-- wheels1 -->
-            <left_joint>rear_left_wheel</left_joint>
-            <right_joint>rear_right_wheel</right_joint>
-            <wheel_separation>${track}</wheel_separation>
-            <wheel_radius>${wheel_radius}</wheel_radius>
-            <odom_publish_frequency>50</odom_publish_frequency>
-            <frame_id>odom</frame_id>
-            <child_frame_id>base_footprint</child_frame_id>
-            <tf_topic>/model/scout_mini/tf_odom</tf_topic>
-        </plugin>
-    </gazebo>
-    <gazebo>
-        <plugin
-            filename="libignition-gazebo-joint-state-publisher-system.so"
-            name="ignition::gazebo::systems::JointStatePublisher">
-            <joint_name>front_right_wheel</joint_name>
-            <topic>/model/scout_mini/joint_states</topic>
-        </plugin>
-        <plugin
-            filename="libignition-gazebo-joint-state-publisher-system.so"
-            name="ignition::gazebo::systems::JointStatePublisher">
-            <joint_name>front_left_wheel</joint_name>
-            <topic>/model/scout_mini/joint_states</topic>
-        </plugin>
-        <plugin
-            filename="libignition-gazebo-joint-state-publisher-system.so"
-            name="ignition::gazebo::systems::JointStatePublisher">
-            <joint_name>rear_right_wheel</joint_name>
-            <topic>/model/scout_mini/joint_states</topic>
-        </plugin>
-        <plugin
-            filename="libignition-gazebo-joint-state-publisher-system.so"
-            name="ignition::gazebo::systems::JointStatePublisher">
-            <joint_name>rear_left_wheel</joint_name>
-            <topic>/model/scout_mini/joint_states</topic>
-        </plugin>
-    </gazebo>
-    <gazebo>
-        <plugin
             filename="ignition-gazebo-pose-publisher-system"
             name="gz::sim::systems::PosePublisher">
@@ -280,3 +256,33 @@
         </plugin>
     </gazebo>
+       <ros2_control name="ScoutMiniGazeboSystem" type="system">
+            <hardware>
+                <plugin>gz_ros2_control/GazeboSimSystem</plugin>
+            </hardware>
+            <joint name="front_left_wheel">
+                <command_interface name="velocity"/>
+                <state_interface name="position"/>
+                <state_interface name="velocity"/>
+            </joint>
+            <joint name="front_right_wheel">
+                <command_interface name="velocity"/>
+                <state_interface name="position"/>
+                <state_interface name="velocity"/>
+            </joint>
+            <joint name="rear_left_wheel">
+                <command_interface name="velocity"/>
+                <state_interface name="position"/>
+                <state_interface name="velocity"/>
+            </joint>
+            <joint name="rear_right_wheel">
+                <command_interface name="velocity"/>
+                <state_interface name="position"/>
+                <state_interface name="velocity"/>
+            </joint>
+        </ros2_control>
+        <gazebo>
+            <plugin filename="libgz_ros2_control-system.so" name="gz_ros2_control::GazeboSimROS2ControlPlugin">
+                <parameters>$(find scout_description)/config/control.yaml</parameters>
+            </plugin>
+        </gazebo>
 </robot>

Commit message: WIP: fixed tf

File: scout_ros2/scout_description/urdf/scout_mini/scout_mini.xacro (robot description, xacro)
@@ -26,21 +26,6 @@
     <xacro:property name="imu_offset_y" value="0"/>
     <xacro:property name="imu_offset_z" value="${-base_z_size/2 + 0.005 + 0.007}"/>
-    <!-- Dummy Root Link -->
-    <link name="dummy_base_link">
-        <!-- No inertial properties for the root link -->
-        <visual>
-            <geometry>
-                <box size="0.001 0.001 0.001" />
-            </geometry>
-            <material name="transparent">
-                <color rgba="0 0 0 0" />
-            </material>
-        </visual>
-        <collision>
-            <geometry>
-                <box size="0.001 0.001 0.001" />
-            </geometry>
-        </collision>
-    </link>
+    <!-- Base Footprint (Root Link) -->
+    <link name="base_footprint"/>
     <!-- Base Link -->
     <link name="base_link">
@@ -63,15 +48,9 @@
         </inertial>
     </link>
-    <!-- Joint connecting dummy_base_link to base_link -->
-    <joint name="dummy_to_base_joint" type="fixed">
-        <parent link="dummy_base_link" />
+    <!-- Joint connecting base_footprint to base_link -->
+    <joint name="base_footprint_to_base_joint" type="fixed">
+        <parent link="base_footprint" />
         <child link="base_link" />
-        <origin xyz="0 0 0" rpy="0 0 0" />
-    </joint>
-    <link name="base_footprint"/>
-    <joint name="base_footprint_joint" type="fixed">
-        <origin xyz="0 0 ${wheel_vertical_offset - wheel_radius}" rpy="0 0 0" />
-        <parent link="base_link" />
-        <child link="base_footprint" />
+        <origin xyz="0 0 ${wheel_radius - wheel_vertical_offset}" rpy="0 0 0" />
     </joint>
     <!-- IMU Sensor -->
@@ -169,5 +148,5 @@
         <origin xyz="${-wheelbase/2} ${-track/2} ${wheel_vertical_offset}" rpy="3.14 0 0" />
     </xacro:scout_mini_wheel>
-    <!-- Gazebo Plugins -->
+    <!-- Gazebo Plugins (Unchanged) -->
     <gazebo reference="imu">
         <sensor name="imu" type="imu">
@@ -256,33 +235,33 @@
         </plugin>
     </gazebo>
-       <ros2_control name="ScoutMiniGazeboSystem" type="system">
-            <hardware>
-                <plugin>gz_ros2_control/GazeboSimSystem</plugin>
-            </hardware>
-            <joint name="front_left_wheel">
-                <command_interface name="velocity"/>
-                <state_interface name="position"/>
-                <state_interface name="velocity"/>
-            </joint>
-            <joint name="front_right_wheel">
-                <command_interface name="velocity"/>
-                <state_interface name="position"/>
-                <state_interface name="velocity"/>
-            </joint>
-            <joint name="rear_left_wheel">
-                <command_interface name="velocity"/>
-                <state_interface name="position"/>
-                <state_interface name="velocity"/>
-            </joint>
-            <joint name="rear_right_wheel">
-                <command_interface name="velocity"/>
-                <state_interface name="position"/>
-                <state_interface name="velocity"/>
-            </joint>
-        </ros2_control>
-        <gazebo>
-            <plugin filename="libgz_ros2_control-system.so" name="gz_ros2_control::GazeboSimROS2ControlPlugin">
-                <parameters>$(find scout_description)/config/control.yaml</parameters>
-            </plugin>
-        </gazebo>
+    <ros2_control name="ScoutMiniGazeboSystem" type="system">
+        <hardware>
+            <plugin>gz_ros2_control/GazeboSimSystem</plugin>
+        </hardware>
+        <joint name="front_left_wheel">
+            <command_interface name="velocity"/>
+            <state_interface name="position"/>
+            <state_interface name="velocity"/>
+        </joint>
+        <joint name="front_right_wheel">
+            <command_interface name="velocity"/>
+            <state_interface name="position"/>
+            <state_interface name="velocity"/>
+        </joint>
+        <joint name="rear_left_wheel">
+            <command_interface name="velocity"/>
+            <state_interface name="position"/>
+            <state_interface name="velocity"/>
+        </joint>
+        <joint name="rear_right_wheel">
+            <command_interface name="velocity"/>
+            <state_interface name="position"/>
+            <state_interface name="velocity"/>
+        </joint>
+    </ros2_control>
+    <gazebo>
+        <plugin filename="libgz_ros2_control-system.so" name="gz_ros2_control::GazeboSimROS2ControlPlugin">
+            <parameters>$(find scout_description)/config/control.yaml</parameters>
+        </plugin>
+    </gazebo>
 </robot>

Commit message: WIP: rotation fix

File: scout_ros2/scout_description/urdf/scout_mini/scout_mini.xacro (robot description, xacro)
@@ -137,5 +137,5 @@
     <!-- Scout wheel macros -->
     <xacro:scout_mini_wheel wheel_prefix="front_right">
-        <origin xyz="${wheelbase/2} ${-track/2} ${wheel_vertical_offset}" rpy="3.14 0 0" />
+        <origin xyz="${wheelbase/2} ${-track/2} ${wheel_vertical_offset}" rpy="0 0 0" />
     </xacro:scout_mini_wheel>
     <xacro:scout_mini_wheel wheel_prefix="front_left">
@@ -146,5 +146,5 @@
     </xacro:scout_mini_wheel>
     <xacro:scout_mini_wheel wheel_prefix="rear_right">
-        <origin xyz="${-wheelbase/2} ${-track/2} ${wheel_vertical_offset}" rpy="3.14 0 0" />
+        <origin xyz="${-wheelbase/2} ${-track/2} ${wheel_vertical_offset}" rpy="0 0 0" />
     </xacro:scout_mini_wheel>
     <!-- Gazebo Plugins (Unchanged) -->

File: scout_ros2/scout_description/urdf/scout_mini/scout_mini_wheel.xacro (robot description, xacro)
@@ -52,5 +52,5 @@
             <child link="${wheel_prefix}_wheel_link"/>
             <xacro:insert_block name="joint_pose"/>
-            <axis xyz="0 -1 0" rpy="0 0 0" />
+            <axis xyz="0 1 0" rpy="0 0 0" />
         </joint>
     </xacro:macro>
